Commit message: Couple the DexHand fingers so they curl, and make the models reproducible
The fingers could not close. Every flexor and DIP was welded, so a finger was
one rigid 75 mm rod on a single hinge and no retargeting could make it grasp.
They are coupled now -- each flexor follows its knuckle, each DIP follows its
flexor -- and one servo curls a whole finger through 163 degrees.

Measured with scripts/motion/analyze_hand.py, welded vs coupled:

                                              welded   coupled
  fingertip travel                            101 mm    137 mm
  closest a fingertip comes to the thumb     85.5 mm   51.8 mm
  ... at the best thumb posture available    43.3 mm    0.0 mm

The last row overturns the earlier finding that this hand cannot pinch: it can,
though not at the thumb posture the config ships, which is joint zero -- the
fully extended splayed pose, 52 mm short of anything. No servo reaches the
thumb, so that posture is a build-time choice; the generator now bakes the
configured angle into the joint origin so setting it actually moves the thumb.

The coupling ratios are estimates. Both ship at 1.0, the right shape for a
linkage-driven finger and the wrong precision, and every number above moves with
them. scripts/motion/fit_finger_coupling.py fits them against the model's own
forward kinematics from measured fingertips; on synthetic data with 0.3 mm of
noise it recovers a 0.83 ratio as 0.824. If this build's fingers really are
rigid, set the multipliers to 0 and regenerate.

Underneath this was a reproducibility problem. generate_urdf.py read the
8-servo description from a path on one developer's laptop when it existed and
the full 16-joint hand when it did not -- two machines, two different robots,
no error either way, and off that laptop the model had no fingertip frames to
aim at. generate_srdf.py had the same dependency and failed outright. The
variant, the fingertip frames and the DexHand SRDF now live in the repository,
and a test regenerates and diffs against what is committed.

Coupling the fingers moved the collision matrices in the safe direction: v1arm
went from 900 disabled pairs to 882, because eighteen pairs that never collided
while the fingers were welded do collide once they curl.

Also fixes an upstream defect the strict mimic check surfaced: all five
<mimic> tags in dexhandv2_right.urdf name their driver without the R_ prefix
the joints carry, so every one points at a joint that does not exist.

Reference for the coupling representation: WIRobotics' ALLEX projects the same
physical relation as a quartic in MJCF and a linear fit in URDF/USD, and
publishes 0.656 for DIP <- PIP on a comparable anthropomorphic finger.

Co-Authored-By: Claude Opus 5 <noreply@anthropic.com>
Claude-Session: https://claude.ai/code/session_01KqSMietALBTZss96WLJWBi

File: ros2_ws/src/berkeley_humanoid_lite_description/urdf/berkeley_humanoid_lite_dexhand.urdf (robot description, URDF)
Before this commit: robot berkeley-humanoid-lite, 42 links, 41 joints
Joints:
- joint R_Index_DIP: axis (none) -> 0.087537 0.996161 -0.000428; limit (none) -> lower=0 upper=0.95 effort=100 velocity=100; mimic (none) -> joint=R_Index_Flexor multiplier=1 offset=0; type fixed -> revolute
- joint R_Index_Flexor: axis (none) -> 0.087537 0.996161 -0.000428; limit (none) -> lower=0 upper=0.95 effort=100 velocity=100; mimic (none) -> joint=R_Index_Pitch multiplier=1 offset=0; type fixed -> revolute
- joint R_Index_Pitch: limit lower=0.0 upper=0.950000 effort=1.5 velocity=3.0 -> lower=0 upper=0.95 effort=100 velocity=100
- joint R_Index_Yaw: limit lower=-0.300000 upper=0.300000 effort=1.5 velocity=3.0 -> lower=-0.3 upper=0.3 effort=100 velocity=100
- joint R_Middle_DIP: axis (none) -> -0.0 1.0 0.0; limit (none) -> lower=0 upper=0.95 effort=100 velocity=100; mimic (none) -> joint=R_Middle_Flexor multiplier=1 offset=0; type fixed -> revolute
- joint R_Middle_Flexor: axis (none) -> -0.0 1.0 0.0; limit (none) -> lower=0 upper=0.95 effort=100 velocity=100; mimic (none) -> joint=R_Middle_Pitch multiplier=1 offset=0; type fixed -> revolute
- joint R_Middle_Pitch: limit lower=0.0 upper=0.950000 effort=1.5 velocity=3.0 -> lower=0 upper=0.95 effort=100 velocity=100
- joint R_Middle_Yaw: limit lower=-0.300000 upper=0.300000 effort=1.5 velocity=3.0 -> lower=-0.3 upper=0.3 effort=100 velocity=100
- joint R_Pinky_DIP: axis (none) -> -0.178318 0.983965 0.003854; limit (none) -> lower=0 upper=0.95 effort=100 velocity=100; mimic (none) -> joint=R_Pinky_Flexor multiplier=1 offset=0; type fixed -> revolute
- joint R_Pinky_Flexor: axis (none) -> -0.178318 0.983965 0.003854; limit (none) -> lower=0 upper=0.95 effort=100 velocity=100; mimic (none) -> joint=R_Pinky_Pitch multiplier=1 offset=0; type fixed -> revolute
- joint R_Pinky_Pitch: limit lower=0.0 upper=0.950000 effort=1.5 velocity=3.0 -> lower=0 upper=0.95 effort=100 velocity=100
- joint R_Pinky_Yaw: limit lower=-0.300000 upper=0.300000 effort=1.5 velocity=3.0 -> lower=-0.3 upper=0.3 effort=100 velocity=100
- joint R_Ring_DIP: axis (none) -> -0.08702 0.996207 -0.00031; limit (none) -> lower=0 upper=0.95 effort=100 velocity=100; mimic (none) -> joint=R_Ring_Flexor multiplier=1 offset=0; type fixed -> revolute
- joint R_Ring_Flexor: axis (none) -> -0.08702 0.996207 -0.00031; limit (none) -> lower=0 upper=0.95 effort=100 velocity=100; mimic (none) -> joint=R_Ring_Pitch multiplier=1 offset=0; type fixed -> revolute
- joint R_Ring_Pitch: limit lower=0.0 upper=0.950000 effort=1.5 velocity=3.0 -> lower=0 upper=0.95 effort=100 velocity=100
- joint R_Ring_Yaw: limit lower=-0.300000 upper=0.300000 effort=1.5 velocity=3.0 -> lower=-0.3 upper=0.3 effort=100 velocity=100

File: ros2_ws/src/berkeley_humanoid_lite_description/urdf/berkeley_humanoid_lite_tuning.urdf (robot description, URDF)
Before this commit: robot berkeley-humanoid-lite, 81 links, 80 joints
Joints:
- joint L_Index_DIP: axis (none) -> -0.087537 0.996161 0.000428; limit (none) -> lower=0 upper=0.95 effort=100 velocity=100; mimic (none) -> joint=L_Index_Flexor multiplier=1 offset=0; type fixed -> revolute
- joint L_Index_Flexor: axis (none) -> -0.087537 0.996161 0.000428; limit (none) -> lower=0 upper=0.95 effort=100 velocity=100; mimic (none) -> joint=L_Index_Pitch multiplier=1 offset=0; type fixed -> revolute
- joint L_Index_Pitch: limit lower=0.0 upper=0.950000 effort=1.5 velocity=3.0 -> lower=0 upper=0.95 effort=100 velocity=100
- joint L_Index_Yaw: limit lower=-0.300000 upper=0.300000 effort=1.5 velocity=3.0 -> lower=-0.3 upper=0.3 effort=100 velocity=100
- joint L_Index_tip_fixed: origin xyz=-0.0011 0.00309 0.0179 rpy=-0 0 -0 -> xyz=-0.0011 -0.00309 0.0179 rpy=0 0 0
- joint L_Middle_DIP: axis (none) -> 0 1 -0; limit (none) -> lower=0 upper=0.95 effort=100 velocity=100; mimic (none) -> joint=L_Middle_Flexor multiplier=1 offset=0; type fixed -> revolute
- joint L_Middle_Flexor: axis (none) -> 0 1 -0; limit (none) -> lower=0 upper=0.95 effort=100 velocity=100; mimic (none) -> joint=L_Middle_Pitch multiplier=1 offset=0; type fixed -> revolute
- joint L_Middle_Pitch: limit lower=0.0 upper=0.950000 effort=1.5 velocity=3.0 -> lower=0 upper=0.95 effort=100 velocity=100
- joint L_Middle_Yaw: limit lower=-0.300000 upper=0.300000 effort=1.5 velocity=3.0 -> lower=-0.3 upper=0.3 effort=100 velocity=100
- joint L_Middle_tip_fixed: origin xyz=-0.0011 0.00309 0.0179 rpy=-0 0 -0 -> xyz=-0.0011 -0.00309 0.0179 rpy=0 0 0
- joint L_Pinky_DIP: axis (none) -> 0.178318 0.983965 -0.003854; limit (none) -> lower=0 upper=0.95 effort=100 velocity=100; mimic (none) -> joint=L_Pinky_Flexor multiplier=1 offset=0; type fixed -> revolute
- joint L_Pinky_Flexor: axis (none) -> 0.178318 0.983965 -0.003854; limit (none) -> lower=0 upper=0.95 effort=100 velocity=100; mimic (none) -> joint=L_Pinky_Pitch multiplier=1 offset=0; type fixed -> revolute
- joint L_Pinky_Pitch: limit lower=0.0 upper=0.950000 effort=1.5 velocity=3.0 -> lower=0 upper=0.95 effort=100 velocity=100
- joint L_Pinky_Yaw: limit lower=-0.300000 upper=0.300000 effort=1.5 velocity=3.0 -> lower=-0.3 upper=0.3 effort=100 velocity=100
- joint L_Pinky_tip_fixed: origin xyz=-0.0011 0.00309 0.0179 rpy=-0 0 -0 -> xyz=-0.0011 -0.00309 0.0179 rpy=0 0 0
- joint L_Ring_DIP: axis (none) -> 0.08702 0.996207 0.00031; limit (none) -> lower=0 upper=0.95 effort=100 velocity=100; mimic (none) -> joint=L_Ring_Flexor multiplier=1 offset=0; type fixed -> revolute
- joint L_Ring_Flexor: axis (none) -> 0.08702 0.996207 0.00031; limit (none) -> lower=0 upper=0.95 effort=100 velocity=100; mimic (none) -> joint=L_Ring_Pitch multiplier=1 offset=0; type fixed -> revolute
- joint L_Ring_Pitch: limit lower=0.0 upper=0.950000 effort=1.5 velocity=3.0 -> lower=0 upper=0.95 effort=100 velocity=100
- joint L_Ring_Yaw: limit lower=-0.300000 upper=0.300000 effort=1.5 velocity=3.0 -> lower=-0.3 upper=0.3 effort=100 velocity=100
- joint L_Ring_tip_fixed: origin xyz=-0.0011 0.00309 0.0179 rpy=-0 0 -0 -> xyz=-0.0011 -0.00309 0.0179 rpy=0 0 0
- joint R_Index_DIP: axis (none) -> 0.087537 0.996161 -0.000428; limit (none) -> lower=0 upper=0.95 effort=100 velocity=100; mimic (none) -> joint=R_Index_Flexor multiplier=1 offset=0; type fixed -> revolute
- joint R_Index_Flexor: axis (none) -> 0.087537 0.996161 -0.000428; limit (none) -> lower=0 upper=0.95 effort=100 velocity=100; mimic (none) -> joint=R_Index_Pitch multiplier=1 offset=0; type fixed -> revolute
- joint R_Index_Pitch: limit lower=0.0 upper=0.950000 effort=1.5 velocity=3.0 -> lower=0 upper=0.95 effort=100 velocity=100
- joint R_Index_Yaw: limit lower=-0.300000 upper=0.300000 effort=1.5 velocity=3.0 -> lower=-0.3 upper=0.3 effort=100 velocity=100
- joint R_Middle_DIP: axis (none) -> -0.0 1.0 0.0; limit (none) -> lower=0 upper=0.95 effort=100 velocity=100; mimic (none) -> joint=R_Middle_Flexor multiplier=1 offset=0; type fixed -> revolute
- joint R_Middle_Flexor: axis (none) -> -0.0 1.0 0.0; limit (none) -> lower=0 upper=0.95 effort=100 velocity=100; mimic (none) -> joint=R_Middle_Pitch multiplier=1 offset=0; type fixed -> revolute
- joint R_Middle_Pitch: limit lower=0.0 upper=0.950000 effort=1.5 velocity=3.0 -> lower=0 upper=0.95 effort=100 velocity=100
- joint R_Middle_Yaw: limit lower=-0.300000 upper=0.300000 effort=1.5 velocity=3.0 -> lower=-0.3 upper=0.3 effort=100 velocity=100
- joint R_Pinky_DIP: axis (none) -> -0.178318 0.983965 0.003854; limit (none) -> lower=0 upper=0.95 effort=100 velocity=100; mimic (none) -> joint=R_Pinky_Flexor multiplier=1 offset=0; type fixed -> revolute
- joint R_Pinky_Flexor: axis (none) -> -0.178318 0.983965 0.003854; limit (none) -> lower=0 upper=0.95 effort=100 velocity=100; mimic (none) -> joint=R_Pinky_Pitch multiplier=1 offset=0; type fixed -> revolute
- joint R_Pinky_Pitch: limit lower=0.0 upper=0.950000 effort=1.5 velocity=3.0 -> lower=0 upper=0.95 effort=100 velocity=100
- joint R_Pinky_Yaw: limit lower=-0.300000 upper=0.300000 effort=1.5 velocity=3.0 -> lower=-0.3 upper=0.3 effort=100 velocity=100
- joint R_Ring_DIP: axis (none) -> -0.08702 0.996207 -0.00031; limit (none) -> lower=0 upper=0.95 effort=100 velocity=100; mimic (none) -> joint=R_Ring_Flexor multiplier=1 offset=0; type fixed -> revolute
- joint R_Ring_Flexor: axis (none) -> -0.08702 0.996207 -0.00031; limit (none) -> lower=0 upper=0.95 effort=100 velocity=100; mimic (none) -> joint=R_Ring_Pitch multiplier=1 offset=0; type fixed -> revolute
- joint R_Ring_Pitch: limit lower=0.0 upper=0.950000 effort=1.5 velocity=3.0 -> lower=0 upper=0.95 effort=100 velocity=100
- joint R_Ring_Yaw: limit lower=-0.300000 upper=0.300000 effort=1.5 velocity=3.0 -> lower=-0.3 upper=0.3 effort=100 velocity=100

File: ros2_ws/src/berkeley_humanoid_lite_description/urdf/berkeley_humanoid_lite_v1arm.urdf (robot description, URDF)
Before this commit: robot berkeley-humanoid-lite, 76 links, 75 joints
Joints:
- joint L_Index_DIP: axis (none) -> -0.087537 0.996161 0.000428; limit (none) -> lower=0 upper=0.95 effort=100 velocity=100; mimic (none) -> joint=L_Index_Flexor multiplier=1 offset=0; type fixed -> revolute
- joint L_Index_Flexor: axis (none) -> -0.087537 0.996161 0.000428; limit (none) -> lower=0 upper=0.95 effort=100 velocity=100; mimic (none) -> joint=L_Index_Pitch multiplier=1 offset=0; type fixed -> revolute
- joint L_Index_Pitch: limit lower=0.0 upper=0.950000 effort=1.5 velocity=3.0 -> lower=0 upper=0.95 effort=100 velocity=100
- joint L_Index_Yaw: limit lower=-0.300000 upper=0.300000 effort=1.5 velocity=3.0 -> lower=-0.3 upper=0.3 effort=100 velocity=100
- joint L_Index_tip_fixed: origin xyz=-0.0011 0.00309 0.0179 rpy=-0 0 -0 -> xyz=-0.0011 -0.00309 0.0179 rpy=0 0 0
- joint L_Middle_DIP: axis (none) -> 0 1 -0; limit (none) -> lower=0 upper=0.95 effort=100 velocity=100; mimic (none) -> joint=L_Middle_Flexor multiplier=1 offset=0; type fixed -> revolute
- joint L_Middle_Flexor: axis (none) -> 0 1 -0; limit (none) -> lower=0 upper=0.95 effort=100 velocity=100; mimic (none) -> joint=L_Middle_Pitch multiplier=1 offset=0; type fixed -> revolute
- joint L_Middle_Pitch: limit lower=0.0 upper=0.950000 effort=1.5 velocity=3.0 -> lower=0 upper=0.95 effort=100 velocity=100
- joint L_Middle_Yaw: limit lower=-0.300000 upper=0.300000 effort=1.5 velocity=3.0 -> lower=-0.3 upper=0.3 effort=100 velocity=100
- joint L_Middle_tip_fixed: origin xyz=-0.0011 0.00309 0.0179 rpy=-0 0 -0 -> xyz=-0.0011 -0.00309 0.0179 rpy=0 0 0
- joint L_Pinky_DIP: axis (none) -> 0.178318 0.983965 -0.003854; limit (none) -> lower=0 upper=0.95 effort=100 velocity=100; mimic (none) -> joint=L_Pinky_Flexor multiplier=1 offset=0; type fixed -> revolute
- joint L_Pinky_Flexor: axis (none) -> 0.178318 0.983965 -0.003854; limit (none) -> lower=0 upper=0.95 effort=100 velocity=100; mimic (none) -> joint=L_Pinky_Pitch multiplier=1 offset=0; type fixed -> revolute
- joint L_Pinky_Pitch: limit lower=0.0 upper=0.950000 effort=1.5 velocity=3.0 -> lower=0 upper=0.95 effort=100 velocity=100
- joint L_Pinky_Yaw: limit lower=-0.300000 upper=0.300000 effort=1.5 velocity=3.0 -> lower=-0.3 upper=0.3 effort=100 velocity=100
- joint L_Pinky_tip_fixed: origin xyz=-0.0011 0.00309 0.0179 rpy=-0 0 -0 -> xyz=-0.0011 -0.00309 0.0179 rpy=0 0 0
- joint L_Ring_DIP: axis (none) -> 0.08702 0.996207 0.00031; limit (none) -> lower=0 upper=0.95 effort=100 velocity=100; mimic (none) -> joint=L_Ring_Flexor multiplier=1 offset=0; type fixed -> revolute
- joint L_Ring_Flexor: axis (none) -> 0.08702 0.996207 0.00031; limit (none) -> lower=0 upper=0.95 effort=100 velocity=100; mimic (none) -> joint=L_Ring_Pitch multiplier=1 offset=0; type fixed -> revolute
- joint L_Ring_Pitch: limit lower=0.0 upper=0.950000 effort=1.5 velocity=3.0 -> lower=0 upper=0.95 effort=100 velocity=100
- joint L_Ring_Yaw: limit lower=-0.300000 upper=0.300000 effort=1.5 velocity=3.0 -> lower=-0.3 upper=0.3 effort=100 velocity=100
- joint L_Ring_tip_fixed: origin xyz=-0.0011 0.00309 0.0179 rpy=-0 0 -0 -> xyz=-0.0011 -0.00309 0.0179 rpy=0 0 0
- joint R_Index_DIP: axis (none) -> 0.087537 0.996161 -0.000428; limit (none) -> lower=0 upper=0.95 effort=100 velocity=100; mimic (none) -> joint=R_Index_Flexor multiplier=1 offset=0; type fixed -> revolute
- joint R_Index_Flexor: axis (none) -> 0.087537 0.996161 -0.000428; limit (none) -> lower=0 upper=0.95 effort=100 velocity=100; mimic (none) -> joint=R_Index_Pitch multiplier=1 offset=0; type fixed -> revolute
- joint R_Index_Pitch: limit lower=0.0 upper=0.950000 effort=1.5 velocity=3.0 -> lower=0 upper=0.95 effort=100 velocity=100
- joint R_Index_Yaw: limit lower=-0.300000 upper=0.300000 effort=1.5 velocity=3.0 -> lower=-0.3 upper=0.3 effort=100 velocity=100
- joint R_Middle_DIP: axis (none) -> -0.0 1.0 0.0; limit (none) -> lower=0 upper=0.95 effort=100 velocity=100; mimic (none) -> joint=R_Middle_Flexor multiplier=1 offset=0; type fixed -> revolute
- joint R_Middle_Flexor: axis (none) -> -0.0 1.0 0.0; limit (none) -> lower=0 upper=0.95 effort=100 velocity=100; mimic (none) -> joint=R_Middle_Pitch multiplier=1 offset=0; type fixed -> revolute
- joint R_Middle_Pitch: limit lower=0.0 upper=0.950000 effort=1.5 velocity=3.0 -> lower=0 upper=0.95 effort=100 velocity=100
- joint R_Middle_Yaw: limit lower=-0.300000 upper=0.300000 effort=1.5 velocity=3.0 -> lower=-0.3 upper=0.3 effort=100 velocity=100
- joint R_Pinky_DIP: axis (none) -> -0.178318 0.983965 0.003854; limit (none) -> lower=0 upper=0.95 effort=100 velocity=100; mimic (none) -> joint=R_Pinky_Flexor multiplier=1 offset=0; type fixed -> revolute
- joint R_Pinky_Flexor: axis (none) -> -0.178318 0.983965 0.003854; limit (none) -> lower=0 upper=0.95 effort=100 velocity=100; mimic (none) -> joint=R_Pinky_Pitch multiplier=1 offset=0; type fixed -> revolute
- joint R_Pinky_Pitch: limit lower=0.0 upper=0.950000 effort=1.5 velocity=3.0 -> lower=0 upper=0.95 effort=100 velocity=100
- joint R_Pinky_Yaw: limit lower=-0.300000 upper=0.300000 effort=1.5 velocity=3.0 -> lower=-0.3 upper=0.3 effort=100 velocity=100
- joint R_Ring_DIP: axis (none) -> -0.08702 0.996207 -0.00031; limit (none) -> lower=0 upper=0.95 effort=100 velocity=100; mimic (none) -> joint=R_Ring_Flexor multiplier=1 offset=0; type fixed -> revolute
- joint R_Ring_Flexor: axis (none) -> -0.08702 0.996207 -0.00031; limit (none) -> lower=0 upper=0.95 effort=100 velocity=100; mimic (none) -> joint=R_Ring_Pitch multiplier=1 offset=0; type fixed -> revolute
- joint R_Ring_Pitch: limit lower=0.0 upper=0.950000 effort=1.5 velocity=3.0 -> lower=0 upper=0.95 effort=100 velocity=100
- joint R_Ring_Yaw: limit lower=-0.300000 upper=0.300000 effort=1.5 velocity=3.0 -> lower=-0.3 upper=0.3 effort=100 velocity=100
