Commit message: Build the hand on the V1 palm, with V2 digits bolted to it
The robot is a DexHand V1 forearm, wrist and palm carrying V2 digit assemblies.
The model had the V1 forearm and wrist right but replaced the whole hand with
V2's, palm included, welded on through an interface part that does not exist.

The V1 palm is four bulk pieces bolted in a row plus a cover plate, and each
digit sits on its own bulk. It is walked out of the description rather than
listed: the palm is whatever hangs off wrist_pitch_upper through *fixed* joints
and the digits hang off it through revolute ones, so following only the fixed
joints separates them without naming either, and an upstream palm redesign
would be picked up rather than missed. The third wrist joint now drives the
first bulk directly, as upstream intends, instead of a bare frame.

Each V2 digit keeps its joint exactly as the variant left it -- axis, travel,
and the mimic tags that make the finger curl -- and takes the V1 mount's origin,
because the bracket it bolts to is V1's. That the two descriptions agree about
where the fingers go is measured, not assumed: referred to a common frame the
four finger mounts differ by 2 to 3 mm. The thumb differs by 15 mm, which is
real -- V2 moved it -- so the adapter is per-digit and the thumb's is called out
as the one that matters.

hand.palm chooses between the two palms; dexhand keeps the V2 one, since a hand
welded straight to an elbow has no V1 wrist to hang a V1 palm off.

The motion package stops assuming the palm is a link called base_link and
derives it as the lowest common ancestor of the finger mounts -- the V2 palm's
one part, or the first bulk of the V1 chain. Four tests measured in the palm
frame and so broke; each is now measured in the finger's own root frame, which
is what they were actually asserting, and the frozen thumb is compared against
upstream rather than against a written-down position.

Vendors the V1 palm meshes for both sides, 15 MB, which the trimmed copy had
dropped on the grounds that the build used V2 fingers -- true of the fingers,
not of the palm they bolt to. SRDFs regenerated: v1arm goes from 882 disabled
pairs to 1318, the palm being five links per side that were not there before.

Co-Authored-By: Claude Opus 5 <noreply@anthropic.com>
Claude-Session: https://claude.ai/code/session_01KqSMietALBTZss96WLJWBi

File: ros2_ws/src/berkeley_humanoid_lite_description/urdf/berkeley_humanoid_lite_tuning.urdf (robot description, URDF)
Before this commit: robot berkeley-humanoid-lite, 81 links, 80 joints
Links:
- removed link L_base_link
- removed link arm_left_wrist_tip
- removed link arm_right_wrist_tip
- removed link base_link
- added link arm_left_hand_cover, mass 0.0276756413; collision mesh filename=package://berkeley_humanoid_lite_description/meshes_v1/left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 scale=0.001 0.001 0.001; visual mesh filename=package://berkeley_humanoid_lite_description/meshes_v1/left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 scale=0.001 0.001 0.001
- added link arm_left_index_bulk, mass 0.0166989673; collision mesh filename=package://berkeley_humanoid_lite_description/meshes_v1/left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 scale=0.001 0.001 0.001; visual mesh filename=package://berkeley_humanoid_lite_description/meshes_v1/left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 scale=0.001 0.001 0.001
- added link arm_left_middle_bulk, mass 0.036646533; collision mesh filename=package://berkeley_humanoid_lite_description/meshes_v1/left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 scale=0.001 0.001 0.001; visual mesh filename=package://berkeley_humanoid_lite_description/meshes_v1/left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 scale=0.001 0.001 0.001
- added link arm_left_pinky_bulk, mass 0.0180357349; collision mesh filename=package://berkeley_humanoid_lite_description/meshes_v1/left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 scale=0.001 0.001 0.001; visual mesh filename=package://berkeley_humanoid_lite_description/meshes_v1/left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 scale=0.001 0.001 0.001
- added link arm_left_ring_bulk, mass 0.0151464713; collision mesh filename=package://berkeley_humanoid_lite_description/meshes_v1/left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 scale=0.001 0.001 0.001; visual mesh filename=package://berkeley_humanoid_lite_description/meshes_v1/left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 scale=0.001 0.001 0.001
- added link arm_right_hand_cover, mass 0.0276756412; collision mesh filename=package://berkeley_humanoid_lite_description/meshes_v1/righ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 scale=0.001 0.001 0.001; visual mesh filename=package://berkeley_humanoid_lite_description/meshes_v1/righ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 scale=0.001 0.001 0.001
- added link arm_right_index_bulk, mass 0.0166988891; collision mesh filename=package://berkeley_humanoid_lite_description/meshes_v1/righ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 scale=0.001 0.001 0.001; visual mesh filename=package://berkeley_humanoid_lite_description/meshes_v1/righ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 scale=0.001 0.001 0.001
- added link arm_right_middle_bulk, mass 0.0366465513; collision mesh filename=package://berkeley_humanoid_lite_description/meshes_v1/righ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 scale=0.001 0.001 0.001; visual mesh filename=package://berkeley_humanoid_lite_description/meshes_v1/righ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 scale=0.001 0.001 0.001
- added link arm_right_pinky_bulk, mass 0.0180357113; collision mesh filename=package://berkeley_humanoid_lite_description/meshes_v1/righ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 scale=0.001 0.001 0.001; visual mesh filename=package://berkeley_humanoid_lite_description/meshes_v1/righ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 scale=0.001 0.001 0.001
- added link arm_right_ring_bulk, mass 0.0151464727; collision mesh filename=package://berkeley_humanoid_lite_description/meshes_v1/righ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 scale=0.001 0.001 0.001; visual mesh filename=package://berkeley_humanoid_lite_description/meshes_v1/righ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 scale=0.001 0.001 0.001
Joints:
- removed joint arm_left_hand_interface
- removed joint arm_right_hand_interface
- added joint arm_left_hand_cover: type fixed, parent arm_left_middle_bulk, child arm_left_hand_cover, origin xyz=0 -0.012 0 rpy=0 0 0
- added joint arm_left_middle_bulk: type fixed, parent arm_left_index_bulk, child arm_left_middle_bulk, origin xyz=-4e-06 -0.006 -0.000452 rpy=0 0 0
- added joint arm_left_pinky_bulk: type fixed, parent arm_left_ring_bulk, child arm_left_pinky_bulk, origin xyz=0 0.006738 0 rpy=0 0 0
- added joint arm_left_ring_bulk: type fixed, parent arm_left_middle_bulk, child arm_left_ring_bulk, origin xyz=0 0.029 0 rpy=0 0 0
- added joint arm_right_hand_cover: type fixed, parent arm_right_middle_bulk, child arm_right_hand_cover, origin xyz=0 0.012 0 rpy=0 0 0
- added joint arm_right_middle_bulk: type fixed, parent arm_right_index_bulk, child arm_right_middle_bulk, origin xyz=0 0.006 0 rpy=0 0 0
- added joint arm_right_pinky_bulk: type fixed, parent arm_right_ring_bulk, child arm_right_pinky_bulk, origin xyz=0 -0.006043 0 rpy=0 0 0
- added joint arm_right_ring_bulk: type fixed, parent arm_right_middle_bulk, child arm_right_ring_bulk, origin xyz=0 -0.029 0 rpy=0 0 0
- joint L_Index_Yaw: origin xyz=0.01778 -0.029123 0.084894 rpy=-0 0 -0 -> xyz=-0.006893 -0.0101 0.084839 rpy=0 0 0; parent L_base_link -> arm_left_index_bulk
- joint L_Middle_Yaw: origin xyz=0.017 -0.00725 0.090983 rpy=-0 0 -0 -> xyz=-0.005866 0.02 0.091 rpy=0 0 0; parent L_base_link -> arm_left_middle_bulk
- joint L_Pinky_Yaw: origin xyz=0.021743 0.035807 0.078606 rpy=-0 0 -0 -> xyz=-0.00427 0.030808 0.078713 rpy=0 0 0; parent L_base_link -> arm_left_pinky_bulk
- joint L_Ring_Yaw: origin xyz=0.018517 0.015063 0.087139 rpy=-0 0 -0 -> xyz=-0.00499 0.015899 0.087076 rpy=0 0 0; parent L_base_link -> arm_left_ring_bulk
- joint L_Thumb_Yaw: origin xyz=0.042207 -0.017744 -0.001358 rpy=-0 0 -0 -> xyz=0.028048 0.005551 0.010472 rpy=0 0 0; parent L_base_link -> arm_left_middle_bulk
- joint R_Index_Yaw: origin xyz=0.01778 0.029123 0.084894 rpy=0 0 0 -> xyz=-0.003905 0.009839 0.084891 rpy=0 0 0; parent base_link -> arm_right_index_bulk
- joint R_Middle_Yaw: origin xyz=0.017 0.00725 0.090983 rpy=0 0 0 -> xyz=-0.002866 -0.02 0.091 rpy=0 0 0; parent base_link -> arm_right_middle_bulk
- joint R_Pinky_Yaw: origin xyz=0.021743 -0.035807 0.078606 rpy=0 0 0 -> xyz=-0.001436 -0.030245 0.078763 rpy=0 0 0; parent base_link -> arm_right_pinky_bulk
- joint R_Ring_Yaw: origin xyz=0.018517 -0.015063 0.087139 rpy=0 0 0 -> xyz=-0.002001 -0.015638 0.087079 rpy=0 0 0; parent base_link -> arm_right_ring_bulk
- joint R_Thumb_Yaw: origin xyz=0.042207 0.017744 -0.001358 rpy=0 0 0 -> xyz=0.026917 -0.00751 0.012735 rpy=0 0 0; parent base_link -> arm_right_middle_bulk
- joint arm_left_wrist_pitch_upper_joint: child arm_left_wrist_tip -> arm_left_index_bulk
- joint arm_right_wrist_pitch_upper_joint: child arm_right_wrist_tip -> arm_right_index_bulk

File: ros2_ws/src/berkeley_humanoid_lite_description/urdf/berkeley_humanoid_lite_v1arm.urdf (robot description, URDF)
Before this commit: robot berkeley-humanoid-lite, 76 links, 75 joints
Links:
- removed link L_base_link
- removed link arm_left_wrist_tip
- removed link arm_right_wrist_tip
- removed link base_link
- added link arm_left_hand_cover, mass 0.0276756413; collision mesh filename=package://berkeley_humanoid_lite_description/meshes_v1/left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 scale=0.001 0.001 0.001; visual mesh filename=package://berkeley_humanoid_lite_description/meshes_v1/left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 scale=0.001 0.001 0.001
- added link arm_left_index_bulk, mass 0.0166989673; collision mesh filename=package://berkeley_humanoid_lite_description/meshes_v1/left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 scale=0.001 0.001 0.001; visual mesh filename=package://berkeley_humanoid_lite_description/meshes_v1/left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 scale=0.001 0.001 0.001
- added link arm_left_middle_bulk, mass 0.036646533; collision mesh filename=package://berkeley_humanoid_lite_description/meshes_v1/left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 scale=0.001 0.001 0.001; visual mesh filename=package://berkeley_humanoid_lite_description/meshes_v1/left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 scale=0.001 0.001 0.001
- added link arm_left_pinky_bulk, mass 0.0180357349; collision mesh filename=package://berkeley_humanoid_lite_description/meshes_v1/left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 scale=0.001 0.001 0.001; visual mesh filename=package://berkeley_humanoid_lite_description/meshes_v1/left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 scale=0.001 0.001 0.001
- added link arm_left_ring_bulk, mass 0.0151464713; collision mesh filename=package://berkeley_humanoid_lite_description/meshes_v1/left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 scale=0.001 0.001 0.001; visual mesh filename=package://berkeley_humanoid_lite_description/meshes_v1/left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 scale=0.001 0.001 0.001
- added link arm_right_hand_cover, mass 0.0276756412; collision mesh filename=package://berkeley_humanoid_lite_description/meshes_v1/righ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 scale=0.001 0.001 0.001; visual mesh filename=package://berkeley_humanoid_lite_description/meshes_v1/righ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 scale=0.001 0.001 0.001
- added link arm_right_index_bulk, mass 0.0166988891; collision mesh filename=package://berkeley_humanoid_lite_description/meshes_v1/righ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 scale=0.001 0.001 0.001; visual mesh filename=package://berkeley_humanoid_lite_description/meshes_v1/righ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 scale=0.001 0.001 0.001
- added link arm_right_middle_bulk, mass 0.0366465513; collision mesh filename=package://berkeley_humanoid_lite_description/meshes_v1/righ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 scale=0.001 0.001 0.001; visual mesh filename=package://berkeley_humanoid_lite_description/meshes_v1/righ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 scale=0.001 0.001 0.001
- added link arm_right_pinky_bulk, mass 0.0180357113; collision mesh filename=package://berkeley_humanoid_lite_description/meshes_v1/righ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 scale=0.001 0.001 0.001; visual mesh filename=package://berkeley_humanoid_lite_description/meshes_v1/righ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 scale=0.001 0.001 0.001
- added link arm_right_ring_bulk, mass 0.0151464727; collision mesh filename=package://berkeley_humanoid_lite_description/meshes_v1/righ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 scale=0.001 0.001 0.001; visual mesh filename=package://berkeley_humanoid_lite_description/meshes_v1/righ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 scale=0.001 0.001 0.001
Joints:
- removed joint arm_left_hand_interface
- removed joint arm_right_hand_interface
- added joint arm_left_hand_cover: type fixed, parent arm_left_middle_bulk, child arm_left_hand_cover, origin xyz=0 -0.012 0 rpy=0 0 0
- added joint arm_left_middle_bulk: type fixed, parent arm_left_index_bulk, child arm_left_middle_bulk, origin xyz=-4e-06 -0.006 -0.000452 rpy=0 0 0
- added joint arm_left_pinky_bulk: type fixed, parent arm_left_ring_bulk, child arm_left_pinky_bulk, origin xyz=0 0.006738 0 rpy=0 0 0
- added joint arm_left_ring_bulk: type fixed, parent arm_left_middle_bulk, child arm_left_ring_bulk, origin xyz=0 0.029 0 rpy=0 0 0
- added joint arm_right_hand_cover: type fixed, parent arm_right_middle_bulk, child arm_right_hand_cover, origin xyz=0 0.012 0 rpy=0 0 0
- added joint arm_right_middle_bulk: type fixed, parent arm_right_index_bulk, child arm_right_middle_bulk, origin xyz=0 0.006 0 rpy=0 0 0
- added joint arm_right_pinky_bulk: type fixed, parent arm_right_ring_bulk, child arm_right_pinky_bulk, origin xyz=0 -0.006043 0 rpy=0 0 0
- added joint arm_right_ring_bulk: type fixed, parent arm_right_middle_bulk, child arm_right_ring_bulk, origin xyz=0 -0.029 0 rpy=0 0 0
- joint L_Index_Yaw: origin xyz=0.01778 -0.029123 0.084894 rpy=-0 0 -0 -> xyz=-0.006893 -0.0101 0.084839 rpy=0 0 0; parent L_base_link -> arm_left_index_bulk
- joint L_Middle_Yaw: origin xyz=0.017 -0.00725 0.090983 rpy=-0 0 -0 -> xyz=-0.005866 0.02 0.091 rpy=0 0 0; parent L_base_link -> arm_left_middle_bulk
- joint L_Pinky_Yaw: origin xyz=0.021743 0.035807 0.078606 rpy=-0 0 -0 -> xyz=-0.00427 0.030808 0.078713 rpy=0 0 0; parent L_base_link -> arm_left_pinky_bulk
- joint L_Ring_Yaw: origin xyz=0.018517 0.015063 0.087139 rpy=-0 0 -0 -> xyz=-0.00499 0.015899 0.087076 rpy=0 0 0; parent L_base_link -> arm_left_ring_bulk
- joint L_Thumb_Yaw: origin xyz=0.042207 -0.017744 -0.001358 rpy=-0 0 -0 -> xyz=0.028048 0.005551 0.010472 rpy=0 0 0; parent L_base_link -> arm_left_middle_bulk
- joint R_Index_Yaw: origin xyz=0.01778 0.029123 0.084894 rpy=0 0 0 -> xyz=-0.003905 0.009839 0.084891 rpy=0 0 0; parent base_link -> arm_right_index_bulk
- joint R_Middle_Yaw: origin xyz=0.017 0.00725 0.090983 rpy=0 0 0 -> xyz=-0.002866 -0.02 0.091 rpy=0 0 0; parent base_link -> arm_right_middle_bulk
- joint R_Pinky_Yaw: origin xyz=0.021743 -0.035807 0.078606 rpy=0 0 0 -> xyz=-0.001436 -0.030245 0.078763 rpy=0 0 0; parent base_link -> arm_right_pinky_bulk
- joint R_Ring_Yaw: origin xyz=0.018517 -0.015063 0.087139 rpy=0 0 0 -> xyz=-0.002001 -0.015638 0.087079 rpy=0 0 0; parent base_link -> arm_right_ring_bulk
- joint R_Thumb_Yaw: origin xyz=0.042207 0.017744 -0.001358 rpy=0 0 0 -> xyz=0.026917 -0.00751 0.012735 rpy=0 0 0; parent base_link -> arm_right_middle_bulk
- joint arm_left_wrist_pitch_upper_joint: child arm_left_wrist_tip -> arm_left_index_bulk
- joint arm_right_wrist_pitch_upper_joint: child arm_right_wrist_tip -> arm_right_index_bulk
